Commit message: finish leg controller

File: new_dog/dog_sim/urdf/big_dog_fixed.SLDASM.urdf (robot description, URDF)
Before this commit: robot dog_sim, 16 links, 15 joints
Links:
- link body: mass 43 -> 10
Joints:
- joint world_joint: origin xyz=0.0 0.0 0.4 rpy=0 0 0 -> xyz=0.0 0.0 0.5 rpy=0 0 0

Commit message: optimize enable

File: new_dog/dog_sim/urdf/big_dog_fixed.SLDASM.urdf (robot description, URDF)
Before this commit: robot dog_sim, 16 links, 15 joints
Joints:
- joint world_joint: origin xyz=0.0 0.0 0.5 rpy=0 0 0 -> xyz=0.0 0.0 0.34 rpy=0 0 0
