Commit message: add locomotion pkg

File: new_dog/dog_sim/urdf/big_dog.SLDASM.urdf (robot description, URDF)
Before this commit: robot new_dog, 15 links, 14 joints
Links:
- link body: mass 43 -> 10; geometry collision mesh filename=package://dog_sim/meshes/body.STL; visual mesh filename=package://dog_sim/meshes/body.STL
- link hokuyo_link: geometry visual mesh filename=package://dog_sim/hokuyo.dae
- link left_back_part_A: geometry collision mesh filename=package://dog_sim/meshes/left_back_part_A.STL; visual mesh filename=package://dog_sim/meshes/left_back_part_A.STL
- link left_back_part_B: geometry collision mesh filename=package://dog_sim/meshes/left_back_part_B.STL; visual mesh filename=package://dog_sim/meshes/left_back_part_B.STL
- link left_back_part_C: geometry collision mesh filename=package://dog_sim/meshes/left_back_part_C.STL; visual mesh filename=package://dog_sim/meshes/left_back_part_C.STL
- link left_front_part_A: geometry collision mesh filename=package://dog_sim/meshes/left_front_part_A.STL; visual mesh filename=package://dog_sim/meshes/left_front_part_A.STL
- link left_front_part_B: geometry collision mesh filename=package://dog_sim/meshes/left_front_part_B.STL; visual mesh filename=package://dog_sim/meshes/left_front_part_B.STL
- link left_front_part_C: geometry collision mesh filename=package://dog_sim/meshes/left_front_part_C.STL; visual mesh filename=package://dog_sim/meshes/left_front_part_C.STL
- link right_back_part_A: geometry collision mesh filename=package://dog_sim/meshes/right_back_part_A.STL; visual mesh filename=package://dog_sim/meshes/right_back_part_A.STL
- link right_back_part_B: geometry collision mesh filename=package://dog_sim/meshes/right_back_part_B.STL; visual mesh filename=package://dog_sim/meshes/right_back_part_B.STL
- link right_back_part_C: geometry collision mesh filename=package://dog_sim/meshes/right_back_part_C.STL; visual mesh filename=package://dog_sim/meshes/right_back_part_C.STL
- link right_front_part_A: geometry collision mesh filename=package://dog_sim/meshes/right_front_part_A.STL; visual mesh filename=package://dog_sim/meshes/right_front_part_A.STL
- link right_front_part_B: geometry collision mesh filename=package://dog_sim/meshes/right_front_part_B.STL; visual mesh filename=package://dog_sim/meshes/right_front_part_B.STL
- link right_front_part_C: geometry collision mesh filename=package://dog_sim/meshes/right_front_part_C.STL; visual mesh filename=package://dog_sim/meshes/right_front_part_C.STL
Joints:
- joint left_front_joint_B: origin xyz=0.0122 0 0.0545 rpy=-0. 1.5708 0 -> xyz=0.0122 0 0.0545 rpy=0 1.5708 0

Commit message: change initial pos& damping factor

File: new_dog/dog_sim/urdf/big_dog.SLDASM.urdf (robot description, URDF)
Before this commit: robot dog_sim, 15 links, 14 joints
Links:
- link left_back_part_A: mass 0.6 -> 0.5
- link left_back_part_B: mass 0.3 -> 0.6
- link left_front_part_A: mass 0.6 -> 0.5
- link left_front_part_B: mass 0.3 -> 0.6
- link right_back_part_A: mass 0.6 -> 0.5
- link right_back_part_B: mass 0.3 -> 0.6
- link right_front_part_A: mass 0.6 -> 0.5
- link right_front_part_B: mass 0.3 -> 0.6

File: new_dog/dog_sim/urdf/big_dog_fixed.SLDASM.urdf (robot description, URDF)
Before this commit: robot dog_sim, 16 links, 15 joints
Links:
- link left_back_part_A: mass 0.6 -> 0.5
- link left_back_part_B: mass 0.3 -> 0.6
- link left_front_part_A: mass 0.6 -> 0.5
- link left_front_part_B: mass 0.3 -> 0.6
- link right_back_part_A: mass 0.6 -> 0.5
- link right_back_part_B: mass 0.3 -> 0.6
- link right_front_part_A: mass 0.6 -> 0.5
- link right_front_part_B: mass 0.3 -> 0.6

Commit message: 该了一下

File: new_dog/dog_sim/urdf/big_dog.SLDASM.urdf (robot description, URDF)
Before this commit: robot dog_sim, 15 links, 14 joints
Links:
- added link camera_link, mass 0.0001; visual mesh filename=package://dog_sim/hokuyo.dae
Joints:
- added joint camerajoint: type fixed, parent body, child camera_link, origin xyz=0.0 -0.255 0.0 rpy=0 0 -1.57
- joint laserjoint: origin xyz=0.0 -0.255 0 rpy=1.5708 0 -1.57 -> xyz=0.0 -0.255 0.1 rpy=0 0 -1.57

File: new_dog/dog_sim/urdf/world.urdf (robot description, URDF)
Before this commit: robot world, 2 links, 1 joints
Links:
- removed link vennue
Joints:
- removed joint joint

Commit message: state_estimation kalman untest

File: new_dog/dog_sim/urdf/big_dog.SLDASM.urdf (robot description, URDF)
Before this commit: robot dog_sim, 16 links, 15 joints
Links:
- added link odom
Joints:
- added joint odomjoint: type fixed, parent body, child odom, origin xyz=0.0 -0.0 -0.05 rpy=0 0 0
